File: doc/pcb/sense/sense.kicad_pcb (KiCad board)
At the start: 2 copper layers, 44 x 42.5 mm, 80 parts, among them J1 PFC24/display, J2 USB_B_Micro, J3 programming, J4 meter, J5 START, J6 SET, J7 RESET, Q1 IRLML0030TR, Q2 BC817, Q3 BC817, Q4 BC817, Q5 BC817, Q6 BC817, Q7 BC817, U1 BME280, U2 STM32G070KB, U3 TC1185-3.3, U4 MCP73831-2-OT, U5 LIS3MDL, Y1 32k768

Commit message: added license
Other:
- net class Default removed
