File: pcb/sense/sense.kicad_sch (KiCad schematic)
At the start: 80 parts, among them J1 PFC24/display, J2 USB_B_Micro, J3 programming, J4 meter, J5 START, J6 SET, J7 RESET, Q1 IRLML0030TR, Q2 BC817, Q3 BC817, Q4 BC817, Q5 BC817, Q6 BC817, Q7 BC817, U1 BME280, U2 STM32G071KxT, U3 TC1185-3.3, U4 MCP73831-2-OT, U5 LIS3MDL, Y1 32k768

Commit message: larger C5
Parts:
- C5: footprint Capacitor_SMD:C_0603_1608Metric -> Capacitor_SMD:C_0805_2012Metric
Changed lines of the file:
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@@
       (effects (font (size 1.27 1.27)) (justify left))
     )
-    (property "Footprint" "Capacitor_SMD:C_0603_1608Metric" (id 2) (at 162.2552 54.61 0)
+    (property "Footprint" "Capacitor_SMD:C_0805_2012Metric" (id 2) (at 162.2552 54.61 0)
       (effects (font (size 1.27 1.27)) hide)
     )
@@
     )
     (path "/00000000-0000-0000-0000-00005dde8678"
-      (reference "C5") (unit 1) (value "475") (footprint "Capacitor_SMD:C_0603_1608Metric")
+      (reference "C5") (unit 1) (value "475") (footprint "Capacitor_SMD:C_0805_2012Metric")
     )
     (path "/00000000-0000-0000-0000-00005de063fb"

Commit message: PCB v1.1
Parts:
- C5: value 475 -> 475 50V
Changed lines of the file:
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@@
       (effects (font (size 1.27 1.27)) (justify left))
     )
-    (property "Value" "475" (id 1) (at 164.211 51.943 0)
+    (property "Value" "475 50V" (id 1) (at 164.211 51.943 0)
       (effects (font (size 1.27 1.27)) (justify left))
     )
@@
     )
     (path "/00000000-0000-0000-0000-00005dde8678"
-      (reference "C5") (unit 1) (value "475") (footprint "Capacitor_SMD:C_0805_2012Metric")
+      (reference "C5") (unit 1) (value "475 50V") (footprint "Capacitor_SMD:C_0805_2012Metric")
     )
     (path "/00000000-0000-0000-0000-00005de063fb"
